Commit message: change urdf format

File: resources/robots/pure/urdf/pure.urdf (robot description, URDF)
Before this commit: robot pure, 21 links, 20 joints
Links:
- link base_link: geometry collision mesh filename=../meshes/base_link.STL; visual mesh filename=../meshes/base_link.STL
- link omni_link_0: geometry collision mesh filename=../meshes/omni_link.STL; visual mesh filename=../meshes/omni_link.STL
- link omni_link_0_roller_link_0: geometry collision mesh filename=../meshes/roller_link_0.STL; visual mesh filename=../meshes/roller_link_0.STL
- link omni_link_0_roller_link_1: geometry collision mesh filename=../meshes/roller_link_1.STL; visual mesh filename=../meshes/roller_link_1.STL
- link omni_link_0_roller_link_2: geometry collision mesh filename=../meshes/roller_link_2.STL; visual mesh filename=../meshes/roller_link_2.STL
- link omni_link_0_roller_link_3: geometry collision mesh filename=../meshes/roller_link_3.STL; visual mesh filename=../meshes/roller_link_3.STL
- link omni_link_1: geometry collision mesh filename=../meshes/omni_link.STL; visual mesh filename=../meshes/omni_link.STL
- link omni_link_1_roller_link_0: geometry collision mesh filename=../meshes/roller_link_0.STL; visual mesh filename=../meshes/roller_link_0.STL
- link omni_link_1_roller_link_1: geometry collision mesh filename=../meshes/roller_link_1.STL; visual mesh filename=../meshes/roller_link_1.STL
- link omni_link_1_roller_link_2: geometry collision mesh filename=../meshes/roller_link_2.STL; visual mesh filename=../meshes/roller_link_2.STL
- link omni_link_1_roller_link_3: geometry collision mesh filename=../meshes/roller_link_3.STL; visual mesh filename=../meshes/roller_link_3.STL
- link omni_link_2: geometry collision mesh filename=../meshes/omni_link.STL; visual mesh filename=../meshes/omni_link.STL
- link omni_link_2_roller_link_0: geometry collision mesh filename=../meshes/roller_link_0.STL; visual mesh filename=../meshes/roller_link_0.STL
- link omni_link_2_roller_link_1: geometry collision mesh filename=../meshes/roller_link_1.STL; visual mesh filename=../meshes/roller_link_1.STL
- link omni_link_2_roller_link_2: geometry collision mesh filename=../meshes/roller_link_2.STL; visual mesh filename=../meshes/roller_link_2.STL
- link omni_link_2_roller_link_3: geometry collision mesh filename=../meshes/roller_link_3.STL; visual mesh filename=../meshes/roller_link_3.STL
- link omni_link_3: geometry collision mesh filename=../meshes/omni_link.STL; visual mesh filename=../meshes/omni_link.STL
- link omni_link_3_roller_link_0: geometry collision mesh filename=../meshes/roller_link_0.STL; visual mesh filename=../meshes/roller_link_0.STL
- link omni_link_3_roller_link_1: geometry collision mesh filename=../meshes/roller_link_1.STL; visual mesh filename=../meshes/roller_link_1.STL
- link omni_link_3_roller_link_2: geometry collision mesh filename=../meshes/roller_link_2.STL; visual mesh filename=../meshes/roller_link_2.STL
- link omni_link_3_roller_link_3: geometry collision mesh filename=../meshes/roller_link_3.STL; visual mesh filename=../meshes/roller_link_3.STL
Joints:
- joint omni_joint_0: limit (none) -> effort=10000 velocity=1000; type continuous -> revolute
- joint omni_joint_1: limit (none) -> effort=10000 velocity=1000; type continuous -> revolute
- joint omni_joint_2: limit (none) -> effort=10000 velocity=1000; type continuous -> revolute
- joint omni_joint_3: limit (none) -> effort=10000 velocity=1000; type continuous -> revolute
